Commit message: v 1.1 changed foot & changed nominal pose

File: rsc/Hop_verParallelAnkleLinks_ver20250304/Hop_verParallelAnkleLinks.urdf (robot description, URDF)
Before this commit: robot DHAL, 11 links, 10 joints
Links:
- link Foot: geometry collision box size=0.24 0.08 0.03; visual mesh filename=URDF_Foot_verHopping1_Simplified.dae scale=1 1 1

Commit message: v 1.1

File: rsc/Hop_verParallelAnkleLinks_ver20250304/Hop_verParallelAnkleLinks.urdf (robot description, URDF)
Before this commit: robot DHAL, 11 links, 10 joints
Links:
- link Foot: mass 1.205532 -> 0.899532
