Commit message: v1.76_bigFoot

File: rsc/Hop_verParallelAnkleLinks_ver20250304/Hop_verParallelAnkleLinks_20250311.urdf (robot description, URDF)
Before this commit: robot DHAL, 11 links, 10 joints
Links:
- link Foot: mass 0.899532 -> 1.0; geometry collision box size=0.26 0.10 0.03; visual mesh filename=URDF_Foot_verHopping1_Simplified.dae scale=1 1 1

Commit message: v1.76_withToe

File: rsc/Hop_verParallelAnkleLinks_ver20250304/Hop_verParallelAnkleLinks_20250311.urdf (robot description, URDF)
Before this commit: robot DHAL, 11 links, 10 joints
Links:
- link Foot: mass 1.0 -> 1.205532; geometry collision box size=0.06 0.1 0.03; collision box size=0.20 0.1 0.03

Commit message: v1.76temp

File: rsc/Hop_verParallelAnkleLinks_ver20250304/Hop_verParallelAnkleLinks_20250311.urdf (robot description, URDF)
Before this commit: robot DHAL, 11 links, 10 joints
Links:
- link Foot: mass 1.205532 -> 0.899532; geometry collision box size=0.24 0.08 0.03; visual mesh filename=URDF_Foot_verHopping1_Simplified.dae scale=1 1 1

Commit message: v1.9 new foot + fine tuning (hard)

File: rsc/Hop_verParallelAnkleLinks_ver20250304/Hop_verParallelAnkleLinks_20250311.urdf (robot description, URDF)
Before this commit: robot DHAL, 11 links, 10 joints
Links:
- link Foot: mass 0.899532 -> 1.0; geometry collision box size=0.265 0.10 0.03; visual mesh filename=URDF_Foot_verHopping1_Simplified.dae scale=1 1 1

Commit message: v 2.2

File: rsc/Hop_verParallelAnkleLinks_ver20250304/Hop_verParallelAnkleLinks_20250311.urdf (robot description, URDF)
Before this commit: robot DHAL, 11 links, 10 joints
Joints:
- joint 00_knee_joint: limit lower=0 upper=2.26893 effort=600.0 velocity=9.0 -> lower=0 upper=2.26893 effort=600.0 velocity=10.11
- joint 07_left_ankle_link_input_joint: limit effort=150.0 velocity=9.0 -> effort=150.0 velocity=18.3
- joint 08_right_ankle_link_input_joint: limit effort=150.0 velocity=9.0 -> effort=150.0 velocity=18.3

Commit message: v2.22 temp with obs normalization -> compare with v2.2

File: rsc/Hop_verParallelAnkleLinks_ver20250304/Hop_verParallelAnkleLinks_20250311.urdf (robot description, URDF)
Before this commit: robot DHAL, 11 links, 10 joints
Links:
- link Foot: mass 1.205532 -> 1.0; geometry collision box size=0.265 0.10 0.03; visual mesh filename=URDF_Foot_verHopping1_Simplified.dae scale=1 1 1

Commit message: v8.0

File: rsc/Hop_verParallelAnkleLinks_ver20250304/Hop_verParallelAnkleLinks_20250311.urdf (robot description, URDF)
Before this commit: robot DHAL, 11 links, 10 joints
Links:
- link Foot: mass 1.0 -> 1.205532; geometry collision box size=0.04 0.1 0.03; collision box size=0.20 0.1 0.03

Commit message: v11.0 -> only backward

File: rsc/Hop_verParallelAnkleLinks_ver20250304/Hop_verParallelAnkleLinks_20250311.urdf (robot description, URDF)
Before this commit: robot DHAL, 11 links, 10 joints
Links:
- link Foot: geometry collision box size=0.055 0.1 0.03; collision box size=0.20 0.1 0.03
