Commit message: urdf foot collision size change 5.5cm > 3.5cm

File: rsc/Hop_verParallelAnkleLinks_ver20250304/Hop_verParallelAnkleLinks_20250311.urdf (robot description, URDF)
Before this commit: robot DHAL, 11 links, 10 joints
Links:
- link Foot: geometry collision box size=0.035 0.1 0.03; collision box size=0.20 0.1 0.03
