Commit message: restitution 0.2 > 0.6 , foot y size 0.1 > 0.08

File: rsc/Hop2_Parallel_Nature_20261001/Hop2_Parallel_Nature_20261001.urdf (robot description, URDF)
Before this commit: robot DHAL, 11 links, 10 joints
Links:
- link Foot: geometry collision box size=0.055 0.08 0.03; collision box size=0.20 0.08 0.03
